File: Hardware/Qwiic_AS3935_Lightning_Detector.sch (EAGLE design)
At the start: 30 parts, among them U1 AS3935

Commit message: Removes old production files, updates board to default to SPI....
* Changes three way jumper to normally open - only need pull ups for I2C mode
* Changes interface select jumper to normally closed (SPI selection)
* Updates notes on both jumpers for these modes
* Removes Qwiic Header
Parts:
- removed J1: (no value), SparkFun-Connectors:QWIIC_CONNECTORJS-1MM
- added R8: 10k, SparkFun-Resistors:10KOHM-0603-1/10W-1%
- JP3: value JUMPER-SMT_2_NO_SILK -> JUMPER-SMT_2_NC_TRACE_SILK; device SparkFun-Jumpers:JUMPER-SMT_2_NO_SILK -> SparkFun-Jumpers:JUMPER-SMT_2_NC_TRACE_SILK
- JP4: value JUMPER-SMT_3_1-NC_TRACE_SILK -> JUMPER-SMT_3_NO_SILK; device SparkFun-Jumpers:JUMPER-SMT_3_1-NC_TRACE_SILK -> SparkFun-Jumpers:JUMPER-SMT_3_NO_SILK
Connections:
- net !CS: now also R8.2
- net 3.3V: no longer J1.2
- net GND: now also R8.1; no longer J1.1
- net MOSI/SDA: no longer J1.3
- net SCLK/SCL: no longer J1.4
Other:
- note added: "Header"
- note added: "Open Jumper to enable I2C"
- note added: "R1 should only closed when there are three or more device on the I2C bus"
- note added: "R2 pullup resistor should be closed if using a single device or more, in I2C mode."
- note added: "v12"
- note removed: "Close Jumper to enable SPI"
- note removed: "Headers"
- note removed: "R1 is disconnected by default and is not recommended unless there are three or more device on the I2C bus"
- note removed: "R2 pullup resistor on the clock is on by default."
- note removed: "v11"
- moved on the sheet: ADD0, ADD1, C1, C2, C3, D1, J4, JP5, L1, R1, R2, R3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
